File: Hardware/voron2_pcb_full/voron2_pcb_full.kicad_pcb (KiCad board)
At the start: 2 copper layers, 143 x 60 mm, 37 parts, among them J1 bme280, J10 y_limit, J11 b_motor, J12 a_motor, J13 hotend_fan, J14 x_limit, J15 Conn_01x03, J16 probe, J17 bme280, J18 extruder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

Commit message: Added Logo And JCLPCB Order Number Location
Parts:
- added G***: LOGO, Logo_footprint:logo_14mm, F.Cu at (98.5, 37.0)
- added G***: LOGO, Logo_footprint:logo_14mm, F.Cu at (135.8, 64.2)
Other:
- board text added: "JLCJLCJLCJLC"
